Commit message: Jazzy & gz8 support
Signed-off-by: Juancams <jc.manzanares.serrano@gmail.com>

File: urdf/gz_waffle.sdf.xacro (robot description, xacro)
@@ -1,4 +1,5 @@
 <?xml version="1.0"?>
-<sdf version="1.6">
+<sdf version="1.6" xmlns:xacro="http://www.ros.org/wiki/xacro">
+    <xacro:arg name="namespace" default=""/>
     <model name="turtlebot3_waffle">
       <pose>0.0 0.0 0.0 0.0 0.0 0.0</pose>
@@ -29,8 +30,11 @@
           <geometry>
             <mesh>
-              <uri>model://turtlebot3_common/meshes/waffle_base.dae</uri>
+              <uri>package://nav2_minimal_tb3_sim/models/turtlebot3_model/meshes/waffle_base.dae</uri>
               <scale>0.001 0.001 0.001</scale>
             </mesh>
           </geometry>
+          <material>
+            <diffuse>1 1 1</diffuse>
+          </material>
         </visual>
       </link>
@@ -39,4 +43,6 @@
           <always_on>true</always_on>
           <update_rate>200</update_rate>
+          <topic>$(arg namespace)/imu</topic>
+          <gz_frame_id>imu_link</gz_frame_id>
           <imu>
             <angular_velocity>
@@ -81,17 +87,9 @@
             </linear_acceleration>
           </imu>
-          <plugin name="turtlebot3_imu" filename="libgazebo_ros_imu_sensor.so">
-            <initial_orientation_as_reference>false</initial_orientation_as_reference>
-            <ros>
-              <!-- <namespace>/tb3</namespace> -->
-              <remapping>~/out:=imu</remapping>
-            </ros>
-          </plugin>
         </sensor>
       </link>
-      <link name="base_mocap">
-        <pose>-0.052 0 0.141 0 0 0</pose>
-        <inertial>
-          <pose>-0.052 0 0.141 0 0 0</pose>
+      <link name="base_scan">
+        <inertial>
+          <pose>-0.064 0 0.121 0 0 0</pose>
           <inertia>
             <ixx>0.001</ixx>
@@ -104,6 +102,6 @@
           <mass>0.125</mass>
         </inertial>
-        <!-- <collision name="mocap_sensor_collision">
-          <pose>-0.052 0 0.160 0 0 0</pose>
+        <collision name="lidar_sensor_collision">
+          <pose>-0.052 0 0.111 0 0 0</pose>
           <geometry>
             <cylinder>
@@ -112,52 +110,24 @@
             </cylinder>
           </geometry>
-        </collision> -->
-        <!-- <visual name="mocap_sensor_visual">
-          <pose>-0.064 0 0.141 0 0 0</pose>
+        </collision>
+        <visual name="lidar_sensor_visual">
+          <pose>-0.064 0 0.121 0 0 0</pose>
           <geometry>
             <mesh>
-              <uri>model://gazebo_mocap_plugin/meshes/rigid_body.dae</uri>
+              <uri>package://nav2_minimal_tb3_sim/models/turtlebot3_model/meshes/lds.dae</uri>
               <scale>0.001 0.001 0.001</scale>
             </mesh>
           </geometry>
-        </visual> -->
-      </link>
-      <link name="base_scan">
-        <pose>-0.052 0 0.121 0 0 0</pose>
-        <inertial>
-          <pose>-0.052 0 0.121 0 0 0</pose>
-          <inertia>
-            <ixx>0.001</ixx>
-            <ixy>0.000</ixy>
-            <ixz>0.000</ixz>
-            <iyy>0.001</iyy>
-            <iyz>0.000</iyz>
-            <izz>0.001</izz>
-          </inertia>
-          <mass>0.125</mass>
-        </inertial>
-        <collision name="lidar_sensor_collision">
-          <pose>-0.052 0 0.131 0 0 0</pose>
-          <geometry>
-            <cylinder>
-              <radius>0.0508</radius>
-              <length>0.055</length>
-            </cylinder>
-          </geometry>
-        </collision>
-        <visual name="lidar_sensor_visual">
-          <pose>-0.064 0 0.131 0 0 0</pose>
-          <geometry>
-            <mesh>
-              <uri>model://turtlebot3_common/meshes/lds.dae</uri>
-              <scale>0.001 0.001 0.001</scale>
-            </mesh>
-          </geometry>
+          <material>
+            <diffuse>1 1 1</diffuse>
+          </material>
         </visual>
-        <sensor name="hls_lfcd_lds" type="ray">
+        <sensor name="hls_lfcd_lds" type="gpu_lidar">
           <always_on>true</always_on>
           <visualize>true</visualize>
-          <pose>-0.064 0 0.131 0 0 0</pose>
+          <pose>-0.064 0 0.15 0 0 0</pose>
           <update_rate>5</update_rate>
+          <topic>$(arg namespace)/scan</topic>
+          <gz_frame_id>base_scan</gz_frame_id>
           <ray>
             <scan>
@@ -170,6 +140,6 @@
             </scan>
             <range>
-              <min>0.120000</min>
-              <max>3.5</max>
+              <min>0.00001</min>
+              <max>20.0</max>
               <resolution>0.015000</resolution>
             </range>
@@ -180,12 +150,4 @@
             </noise>
           </ray>
-          <plugin name="turtlebot3_laserscan" filename="libgazebo_ros_ray_sensor.so">
-            <ros>
-                <!-- <namespace>/tb3</namespace> -->
-                <remapping>~/out:=scan</remapping>
-            </ros>
-            <output_type>sensor_msgs/LaserScan</output_type>
-            <frame_name>base_scan</frame_name>
-          </plugin>
         </sensor>
       </link>
@@ -212,12 +174,11 @@
           </geometry>
           <surface>
-            <!-- This friction pamareter don't contain reliable data!! -->
             <friction>
               <ode>
-                <mu>100000.0</mu>
-                <mu2>100000.0</mu2>
-                <fdir1>0 0 0</fdir1>
-                <slip1>0.0</slip1>
-                <slip2>0.0</slip2>
+                <mu>1</mu>
+                <mu2>1</mu2>
+                <slip1>0.035</slip1>
+                <slip2>0</slip2>
+                <fdir1>0 0 1</fdir1>
               </ode>
             </friction>
@@ -238,8 +199,11 @@
           <geometry>
             <mesh>
-              <uri>model://turtlebot3_common/meshes/tire.dae</uri>
+              <uri>package://nav2_minimal_tb3_sim/models/turtlebot3_model/meshes/tire.dae</uri>
               <scale>0.001 0.001 0.001</scale>
             </mesh>
           </geometry>
+          <material>
+            <diffuse>1 1 1</diffuse>
+          </material>
         </visual>
       </link>
@@ -266,12 +230,11 @@
           </geometry>
           <surface>
-            <!-- This friction pamareter don't contain reliable data!! -->
             <friction>
               <ode>
-                <mu>100000.0</mu>
-                <mu2>100000.0</mu2>
-                <fdir1>0 0 0</fdir1>
-                <slip1>0.0</slip1>
-                <slip2>0.0</slip2>
+                <mu>1</mu>
+                <mu2>1</mu2>
+                <slip1>0.035</slip1>
+                <slip2>0</slip2>
+                <fdir1>0 0 1</fdir1>
               </ode>
             </friction>
@@ -292,8 +255,11 @@
           <geometry>
             <mesh>
-              <uri>model://turtlebot3_common/meshes/tire.dae</uri>
+              <uri>package://nav2_minimal_tb3_sim/models/turtlebot3_model/meshes/tire.dae</uri>
               <scale>0.001 0.001 0.001</scale>
             </mesh>
           </geometry>
+          <material>
+            <diffuse>1 1 1</diffuse>
+          </material>
         </visual>
       </link>
@@ -365,5 +331,4 @@
       </link>
       <link name="camera_link">
-        <pose>0.069 -0.047 0.107 0 0 0</pose>
         <inertial>
           <pose>0.069 -0.047 0.107 0 0 0</pose>
@@ -391,25 +356,26 @@
           <update_rate>5</update_rate>
           <pose>0.064 -0.047 0.107 0 0 0</pose>
+          <gz_frame_id>camera_depth_frame</gz_frame_id>
           <camera name="realsense_depth_camera">
+            <horizontal_fov>1.047</horizontal_fov>
+            <image>
+              <width>320</width>
+              <height>240</height>
+            </image>
+            <lens>
+              <projection>
+                <!-- focal_length = fx = fy = width / ( 2 * tan (hfov / 2 ) ) -->
+                <!-- tx = hackBaseline * focal_length -->
+                <tx>19.4</tx>
+              </projection>
+            </lens>
+            <depth_camera>
+              <clip>
+                <near>0.001</near>
+                <far>5.0</far>
+              </clip>
+            </depth_camera>
           </camera>
-          <plugin name="intel_realsense_r200_depth_driver" filename="libgazebo_ros_camera.so">
-            <ros>
-            </ros>
-            <camera_name>intel_realsense_r200_depth</camera_name>
-            <frame_name>camera_depth_frame</frame_name>
-            <hack_baseline>0.07</hack_baseline>
-            <min_depth>0.001</min_depth>
-            <max_depth>5.0</max_depth>
-          </plugin>
         </sensor>
-        <collision name="collision">
-          <pose>0 0.047 -0.005 0 0 0</pose>
-          <geometry>
-            <box>
-              <size>0.008 0.130 0.022</size>
-            </box>
-          </geometry>
-        </collision>
-        <pose>0.069 -0.047 0.107 0 0 0</pose>
       </link>
       <joint name="base_joint" type="fixed">
@@ -442,12 +408,4 @@
         <child>caster_back_left_link</child>
       </joint>
-      <joint name="mocap_joint" type="fixed">
-        <parent>base_link</parent>
-        <child>base_mocap</child>
-        <pose>-0.064 0 0.141 0 0 0</pose>
-        <axis>
-          <xyz>0 0 1</xyz>
-        </axis>
-      </joint>
       <joint name="lidar_joint" type="fixed">
         <parent>base_link</parent>
@@ -466,53 +424,39 @@
         </axis>
       </joint>
-      <joint name="camera_rgb_joint" type="fixed">
-        <parent>camera_link</parent>
-        <child>camera_rgb_frame</child>
-        <pose>0.005 0.018 0.013 0 0 0</pose>
-        <axis>
-          <xyz>0 0 1</xyz>
-        </axis>
-      </joint>
-      <plugin name="turtlebot3_diff_drive" filename="libgazebo_ros_diff_drive.so">
-        <ros>
-          <!-- <namespace>/tb3</namespace> -->
-          <!--since gazebo_plugins publish tf topic in global namespace /tf only and it
-            cannot be remapped like (namespace/tf) through launch arguments -->
-          <remapping>/tf:=tf</remapping>
-        </ros>
-        <update_rate>30</update_rate>
-        <!-- wheels -->
+      <plugin
+        filename="gz-sim-diff-drive-system"
+        name="gz::sim::systems::DiffDrive">
         <left_joint>wheel_left_joint</left_joint>
         <right_joint>wheel_right_joint</right_joint>
-        <!-- kinematics -->
         <wheel_separation>0.287</wheel_separation>
-        <wheel_diameter>0.066</wheel_diameter>
-        <!-- limits -->
-        <max_wheel_torque>20</max_wheel_torque>
-        <max_wheel_acceleration>1.0</max_wheel_acceleration>
-        <command_topic>cmd_vel</command_topic>
-        <!-- output -->
-        <publish_odom>true</publish_odom>
-        <publish_odom_tf>true</publish_odom_tf>
-        <publish_wheel_tf>false</publish_wheel_tf>
-        <odometry_topic>odom</odometry_topic>
-        <odometry_frame>odom</odometry_frame>
-        <robot_base_frame>base_footprint</robot_base_frame>
+        <wheel_radius>0.033</wheel_radius>
+        <max_linear_acceleration>1</max_linear_acceleration>
+        <min_linear_acceleration>-1</min_linear_acceleration>
+        <max_angular_acceleration>2</max_angular_acceleration>
+        <min_angular_acceleration>-2</min_angular_acceleration>
+        <max_linear_velocity>0.46</max_linear_velocity>
+        <min_linear_velocity>-0.46</min_linear_velocity>
+        <max_angular_velocity>1.9</max_angular_velocity>
+        <min_angular_velocity>-1.9</min_angular_velocity>
+        <topic>$(arg namespace)/cmd_vel</topic>
+        <odom_topic>$(arg namespace)/odom</odom_topic>
+        <tf_topic>$(arg namespace)/tf</tf_topic>
+        <frame_id>odom</frame_id>
+        <child_frame_id>base_footprint</child_frame_id>
+        <odom_publish_frequency>30</odom_publish_frequency>
       </plugin>
-      <plugin name="turtlebot3_joint_state" filename="libgazebo_ros_joint_state_publisher.so">
-        <ros>
-          <!-- <namespace>/tb3</namespace> -->
-            <remapping>~/out:=joint_states</remapping>
-        </ros>
-        <update_rate>30</update_rate>
+      <plugin
+        filename="gz-sim-joint-state-publisher-system"
+        name="gz::sim::systems::JointStatePublisher">
         <joint_name>wheel_left_joint</joint_name>
         <joint_name>wheel_right_joint</joint_name>
+        <topic>$(arg namespace)/joint_states</topic>
+        <update_rate>30</update_rate>
       </plugin>
-      <plugin name="gazebo_ros_mocap" filename="libgazebo_ros_mocap.so">
-        <rigid_link>base_link</rigid_link>
-        <rigid_link>base_mocap</rigid_link>
-        <marker_link>camera_link</marker_link>
+      <plugin
+        filename="libgz_ros_mocap.so"
+        name="gz::sim::systems::GzRosMocap">
         <rigid_link>base_footprint</rigid_link>
-      </plugin>
+    </plugin>
     </model>
 </sdf>
